File: Keyboard/MyOwnKeyboard.sch (KiCad schematic (older format))
At the start: 465 parts, among them J1 Mini-DIN-6, Q1 RFD14N05L, SW1 SW_SPST, SW10 SW_SPST, SW100 SW_SPST, SW101 SW_SPST, SW102 SW_SPST, SW103 SW_SPST, SW104 SW_SPST, SW105 SW_SPST, SW106 SW_SPST, SW107 SW_SPST, SW108 SW_SPST, SW109 SW_SPST, SW11 SW_SPST, SW110 SW_SPST, SW111 SW_SPST, SW112 SW_SPST, SW113 SW_SPST, SW114 SW_SPST, SW12 SW_SPST, SW13 SW_SPST, SW14 SW_SPST, SW15 SW_SPST, SW16 SW_SPST, SW17 SW_SPST, SW18 SW_SPST, SW19 SW_SPST, SW2 SW_SPST, SW20 SW_SPST, SW21 SW_SPST, SW22 SW_SPST, SW23 SW_SPST, SW24 SW_SPST, SW25 SW_SPST, SW26 SW_SPST, SW27 SW_SPST, SW28 SW_SPST, SW29 SW_SPST, SW3 SW_SPST, SW30 SW_SPST, SW31 SW_SPST, SW32 SW_SPST, SW33 SW_SPST, SW34 SW_SPST, SW35 SW_SPST, SW36 SW_SPST, SW37 SW_SPST, SW38 SW_SPST, SW39 SW_SPST, SW4 SW_SPST, SW40 SW_SPST, SW41 SW_SPST, SW42 SW_SPST, SW43 SW_SPST, SW44 SW_SPST, SW45 SW_SPST, SW46 SW_SPST, SW47 SW_SPST, SW48 SW_SPST, SW49 SW_SPST, SW5 SW_SPST, SW50 SW_SPST, SW51 SW_SPST, SW52 SW_SPST, SW53 SW_SPST, SW54 SW_SPST, SW55 SW_SPST, SW56 SW_SPST, SW57 SW_SPST, SW58 SW_SPST, SW59 SW_SPST, SW6 SW_SPST, SW60 SW_SPST, SW61 SW_SPST, SW62 SW_SPST, SW63 SW_SPST, SW64 SW_SPST, SW65 SW_SPST, SW66 SW_SPST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

Commit message: Add function key
Parts:
- added RN? (x2): R_Network08, Resistor_THT:R_Array_SIP9, symbol Device:R_Network08
- added RN?: R_Network03, Resistor_THT:R_Array_SIP4, symbol Device:R_Network03
Connections:
- wire segments 1199 -> 1264
Other:
- moved on the sheet: D229, D230, J1, R117, R118
