File: Keyboard/MyOwnKeyboard.kicad_pcb (KiCad board)
At the start: 2 copper layers, 466 parts, among them J1 Mini-DIN-6, J2 ISP Header, Q1 2N7000, SW1 SW_SPST, SW10 SW_SPST, SW100 SW_SPST, SW101 SW_SPST, SW102 SW_SPST, SW103 SW_SPST, SW104 SW_SPST, SW105 SW_SPST, SW106 SW_SPST, SW107 SW_SPST, SW108 SW_SPST, SW109 SW_SPST, SW11 SW_SPST, SW110 SW_SPST, SW111 SW_SPST, SW112 SW_SPST, SW113 SW_SPST, SW114 SW_SPST, SW12 SW_SPST, SW13 SW_SPST, SW14 SW_SPST, SW15 SW_SPST, SW16 SW_SPST, SW17 SW_SPST, SW18 SW_SPST, SW19 SW_SPST, SW2 SW_SPST, SW20 SW_SPST, SW21 SW_SPST, SW22 SW_SPST, SW23 SW_SPST, SW24 SW_SPST, SW25 SW_SPST, SW26 SW_SPST, SW27 SW_SPST, SW28 SW_SPST, SW29 SW_SPST, SW3 SW_SPST, SW30 SW_SPST, SW31 SW_SPST, SW32 SW_SPST, SW33 SW_SPST, SW34 SW_SPST, SW35 SW_SPST, SW36 SW_SPST, SW37 SW_SPST, SW38 SW_SPST, SW39 SW_SPST, SW4 SW_SPST, SW40 SW_SPST, SW41 SW_SPST, SW42 SW_SPST, SW43 SW_SPST, SW44 SW_SPST, SW45 SW_SPST, SW46 SW_SPST, SW47 SW_SPST, SW48 SW_SPST, SW49 SW_SPST, SW5 SW_SPST, SW50 SW_SPST, SW51 SW_SPST, SW52 SW_SPST, SW53 SW_SPST, SW54 SW_SPST, SW55 SW_SPST, SW56 SW_SPST, SW57 SW_SPST, SW58 SW_SPST, SW59 SW_SPST, SW6 SW_SPST, SW60 SW_SPST, SW61 SW_SPST, SW62 SW_SPST, SW63 SW_SPST, SW64 SW_SPST, SW65 SW_SPST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

Commit message: Initial layout
Parts:
- removed D1, D104, D105, D11, D19, D2, D3, D38, D4, D57, D76, D93, D95: 1N4148, Diode_SMD:D_MiniMELF
- removed D115, D116, D117, D118, D125, D133, D152, D171, D190, D207, D209, D218, D219: LED, MyOwnKeyboard:158301250
- removed R106, R107, R13, R21, R3, R4, R40, R5, R59, R6, R78, R95, R97: 2.26k, Resistor_SMD:R_0805_2012Metric_Pad1.15x1.40mm_HandSolder
- removed SW1, SW104, SW105, SW11, SW19, SW2, SW3, SW38, SW4, SW57, SW76, SW93, SW95: SW_SPST, MyOwnKeyboard:SW_Cherry_MX_1.00u_PCB
- added M1: MountingHole_2.7mm_M2.5_Pad_Via, MountingHole:MountingHole_2.7mm_M2.5_Pad_Via, F.Cu at (30.9, 175.8)
- added M10: MountingHole_2.7mm_M2.5_Pad_Via, MountingHole:MountingHole_2.7mm_M2.5_Pad_Via, F.Cu at (199.5, 289.8)
- added M11: MountingHole_2.7mm_M2.5_Pad_Via, MountingHole:MountingHole_2.7mm_M2.5_Pad_Via, F.Cu at (201.9, 220.9)
- added M12: MountingHole_2.7mm_M2.5_Pad_Via, MountingHole:MountingHole_2.7mm_M2.5_Pad_Via, F.Cu at (237.5, 257.1)
- added M13: MountingHole_2.7mm_M2.5_Pad_Via, MountingHole:MountingHole_2.7mm_M2.5_Pad_Via, F.Cu at (270.8, 289.8)
- added M14: MountingHole_2.7mm_M2.5_Pad_Via, MountingHole:MountingHole_2.7mm_M2.5_Pad_Via, F.Cu at (280.2, 219.3)
- added M15: MountingHole_2.7mm_M2.5_Pad_Via, MountingHole:MountingHole_2.7mm_M2.5_Pad_Via, F.Cu at (294.5, 175.8)
- added M16: MountingHole_2.7mm_M2.5_Pad_Via, MountingHole:MountingHole_2.7mm_M2.5_Pad_Via, F.Cu at (323.0, 255.8)
- added M17: MountingHole_2.7mm_M2.5_Pad_Via, MountingHole:MountingHole_2.7mm_M2.5_Pad_Via, F.Cu at (356.2, 219.3)
- added M18: MountingHole_2.7mm_M2.5_Pad_Via, MountingHole:MountingHole_2.7mm_M2.5_Pad_Via, F.Cu at (365.8, 289.8)
- added M19: MountingHole_2.7mm_M2.5_Pad_Via, MountingHole:MountingHole_2.7mm_M2.5_Pad_Via, F.Cu at (380.0, 175.8)
- added M2: MountingHole_2.7mm_M2.5_Pad_Via, MountingHole:MountingHole_2.7mm_M2.5_Pad_Via, F.Cu at (30.9, 232.8)
- added M20: MountingHole_2.7mm_M2.5_Pad_Via, MountingHole:MountingHole_2.7mm_M2.5_Pad_Via, F.Cu at (413.2, 273.1)
- added M21: MountingHole_2.7mm_M2.5_Pad_Via, MountingHole:MountingHole_2.7mm_M2.5_Pad_Via, F.Cu at (434.6, 220.9)
- added M22: MountingHole_2.7mm_M2.5_Pad_Via, MountingHole:MountingHole_2.7mm_M2.5_Pad_Via, F.Cu at (463.1, 175.8)
- added M23: MountingHole_2.7mm_M2.5_Pad_Via, MountingHole:MountingHole_2.7mm_M2.5_Pad_Via, F.Cu at (463.1, 232.8)
- added M24: MountingHole_2.7mm_M2.5_Pad_Via, MountingHole:MountingHole_2.7mm_M2.5_Pad_Via, F.Cu at (463.1, 289.8)
- added M3: MountingHole_2.7mm_M2.5_Pad_Via, MountingHole:MountingHole_2.7mm_M2.5_Pad_Via, F.Cu at (30.9, 289.8)
- added M4: MountingHole_2.7mm_M2.5_Pad_Via, MountingHole:MountingHole_2.7mm_M2.5_Pad_Via, F.Cu at (71.2, 218.5)
- added M5: MountingHole_2.7mm_M2.5_Pad_Via, MountingHole:MountingHole_2.7mm_M2.5_Pad_Via, F.Cu at (71.2, 256.5)
- added M6: MountingHole_2.7mm_M2.5_Pad_Via, MountingHole:MountingHole_2.7mm_M2.5_Pad_Via, F.Cu at (133.0, 218.5)
- added M7: MountingHole_2.7mm_M2.5_Pad_Via, MountingHole:MountingHole_2.7mm_M2.5_Pad_Via, F.Cu at (113.2, 289.8)
- added M8: MountingHole_2.7mm_M2.5_Pad_Via, MountingHole:MountingHole_2.7mm_M2.5_Pad_Via, F.Cu at (173.4, 175.8)
- added M9: MountingHole_2.7mm_M2.5_Pad_Via, MountingHole:MountingHole_2.7mm_M2.5_Pad_Via, F.Cu at (180.5, 251.8)
- D229, D230: footprint MyOwnKeyboard:158301250 -> MyOwnKeyboard:158301250_Face_Down; moved to B.Cu
- J2, Q1, R1, R2: moved to B.Cu
- SW101, SW102, SW103, SW111, SW112, SW113: footprint MyOwnKeyboard:SW_Cherry_MX_1.00u_PCB -> MyOwnKeyboard:SW_Cherry_MX_1.25u_PCB
- SW108: footprint MyOwnKeyboard:SW_Cherry_MX_1.00u_PCB -> MyOwnKeyboard:SW_Cherry_MX_7.00u_PCB
- SW114, SW82: footprint MyOwnKeyboard:SW_Cherry_MX_1.00u_PCB -> MyOwnKeyboard:SW_Cherry_MX_2.25u_PCB
- SW45, SW94: footprint MyOwnKeyboard:SW_Cherry_MX_1.00u_PCB -> MyOwnKeyboard:SW_Cherry_MX_1.50u_PCB
- SW61, SW80: footprint MyOwnKeyboard:SW_Cherry_MX_1.00u_PCB -> MyOwnKeyboard:SW_Cherry_MX_2.00u_Vertical_PCB
- SW63: footprint MyOwnKeyboard:SW_Cherry_MX_1.00u_PCB -> MyOwnKeyboard:SW_Cherry_MX_1.75u_PCB
- SW75: footprint MyOwnKeyboard:SW_Cherry_MX_1.00u_PCB -> MyOwnKeyboard:SW_Cherry_MX_2.00u_PCB
- SW92: footprint MyOwnKeyboard:SW_Cherry_MX_1.00u_PCB -> MyOwnKeyboard:SW_Cherry_MX_2.75u_PCB
- U1: footprint Package_DIP:DIP-40_W15.24mm -> Package_DIP:DIP-40_W15.24mm_Socket
- moved D230 183.8 mm to (104.9, 189.8)
- moved R118 180.7 mm to (110.3, 189.8), turned to 180 degrees
- moved D229 174.9 mm to (105.8, 185.5)
- moved R117 172.0 mm to (111.2, 185.5), turned to 180 degrees
- moved R2 158.7 mm to (162.3, 184.5), turned to 270 degrees
- moved R1 157.9 mm to (162.3, 180.7), turned to 270 degrees
- moved Q1 152.5 mm to (166.1, 181.2), turned to 270 degrees
- moved D206 144.5 mm to (434.6, 261.0)
- moved SW92 144.5 mm to (434.6, 266.0)
- moved D92 144.5 mm to (442.6, 266.8)
- moved R94 144.5 mm to (434.8, 261.2)
- moved J2 144.3 mm to (158.7, 179.8), turned to 180 degrees
- moved J1 140.8 mm to (204.5, 177.2)
- moved U1 134.2 mm to (119.4, 189.9)
- moved D205 132.6 mm to (399.0, 261.0)
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Connections:
- U1 pad 25: (no net) -> Earth
Routing:
- net 5v: track 0.00 -> 2688.9 mm, vias 0 -> 10
- net Net-(D115-Pad1): track 0.00 -> 2618.3 mm, vias 0 -> 111
- net P: track 0.00 -> 465.8 mm, vias 0 -> 2
- net R: track 0.00 -> 462.8 mm, vias 0 -> 4
- net Q: track 0.00 -> 415.6 mm, vias 0 -> 2
- net MISO: track 0.00 -> 398.3 mm, vias 0 -> 2
- net MOSI: track 0.00 -> 381.8 mm, vias 0 -> 2
- net S: track 0.00 -> 373.6 mm
- net M: track 0.00 -> 348.8 mm, vias 0 -> 2
- net G: track 0.00 -> 338.2 mm, vias 0 -> 2
- net L: track 0.00 -> 311.6 mm, vias 0 -> 2
- net H: track 0.00 -> 306.7 mm, vias 0 -> 2
- net F: track 0.00 -> 272.5 mm
- net I: track 0.00 -> 268.5 mm, vias 0 -> 2
- net J: track 0.00 -> 268.4 mm, vias 0 -> 2
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Other:
- board outline added: 441.8 x 123.5 mm

Commit message: Finalise routing
Routing:
- net 5: track 207.5 -> 718.9 mm, vias 2 -> 12
- net 6: track 229.4 -> 731.6 mm, vias 2 -> 6
- net 4: track 184.6 -> 682.9 mm, vias 2 -> 9
- net 2: track 140.5 -> 585.2 mm, vias 0 -> 6
- net 3: track 162.7 -> 593.4 mm, vias 2 -> 8
- net 1: track 86.2 -> 336.4 mm
- net I: track 268.5 -> 269.7 mm
- net E: track 196.9 -> 197.9 mm
- net Earth: vias 17 -> 34

Commit message: Finalise board for production
Removed most silkscreen footprint references for switches, diodes, and resistors
Added a legend for the ISP header
Filled in as much ground as possible
Routing:
- net Earth: vias 34 -> 57
Other:
- board text added: "5v"
- board text added: "CLK"
- board text added: "GND"
- board text added: "MISO"
- board text added: "MOSI"
- board text added: "RST"

Commit message: Finalise revision 1 design
Parts:
- J1: moved to B.Cu
- moved J1 0.44 mm to (204.5, 177.6), turned to 0 degrees
Routing:
- net /Data: track 68.1 -> 76.5 mm
- net /Clk: track 61.1 -> 67.4 mm
- net 5v: track 2688.9 -> 2693.7 mm
- net 1: track 336.4 -> 334.7 mm
- net G: track 338.2 -> 336.5 mm
- net Earth: vias 57 -> 60
Other:
- board text added: "Contains"
- board text added: "Design finalised: 2021-06-15"
- board text added: "Designed in Australia"
- board text added: "JLC Order No.: JLCJLCJLCJLC"
- board text added: "Lead"
- board text added: "Revision 1"
- board text added: "The Thomotron Custom"
- board text added: "github.com/thomotron/keyboard"
