File: TestKeypad/TestKeypad.sch (KiCad schematic (older format))
At the start: 73 parts, among them J1 Mini-DIN-6, J2 ISP Header, Q1 2N7000, SW1 SW_SPST, SW10 SW_SPST, SW11 SW_SPST, SW12 SW_SPST, SW13 SW_SPST, SW14 SW_SPST, SW15 SW_SPST, SW16 SW_SPST, SW2 SW_SPST, SW3 SW_SPST, SW4 SW_SPST, SW5 SW_SPST, SW6 SW_SPST, SW7 SW_SPST, SW8 SW_SPST, SW9 SW_SPST, U1 ATmega8535-16PU

Commit message: Update keypad also
Parts:
- removed RN1: 100k, Resistor_THT:R_Array_SIP9, symbol Device:R_Network08
- D17, D18, D19, D20, D21, D22, D23, D24, D25, D26, D27, D28, D29, D30, D31, D32: footprint Diode_SMD:D_MiniMELF_Handsoldering -> Diode_SMD:D_MiniMELF
Connections:
- net A: now also D17.2 (A), D21.2 (A), D25.2 (A), D29.2 (A); no longer D17.1 (K), D21.1 (K), D25.1 (K), D29.1 (K)
- net B: now also D18.2 (A), D22.2 (A), D26.2 (A), D30.2 (A); no longer D18.1 (K), D22.1 (K), D26.1 (K), D30.1 (K)
- net C: now also D19.2 (A), D23.2 (A), D27.2 (A), D31.2 (A); no longer D19.1 (K), D23.1 (K), D27.1 (K), D31.1 (K)
- net D: now also D20.2 (A), D24.2 (A), D28.2 (A), D32.2 (A); no longer D20.1 (K), D24.1 (K), D28.1 (K), D32.1 (K)
- net at SW1.2 (B): now also D17.1 (K); no longer D17.2 (A)
- net at SW5.2 (B): now also D21.1 (K); no longer D21.2 (A)
- net at SW9.2 (B): now also D25.1 (K); no longer D25.2 (A)
- net at SW13.2 (B): now also D29.1 (K); no longer D29.2 (A)
- net at SW2.2 (B): now also D18.1 (K); no longer D18.2 (A)
- net at SW6.2 (B): now also D22.1 (K); no longer D22.2 (A)
- net at SW10.2 (B): now also D26.1 (K); no longer D26.2 (A)
- net at SW14.2 (B): now also D30.1 (K); no longer D30.2 (A)
- net at SW3.2 (B): now also D19.1 (K); no longer D19.2 (A)
- net at SW7.2 (B): now also D23.1 (K); no longer D23.2 (A)
- net at SW11.2 (B): now also D27.1 (K); no longer D27.2 (A)
- net at SW15.2 (B): now also D31.1 (K); no longer D31.2 (A)
- net at SW4.2 (B): now also D20.1 (K); no longer D20.2 (A)
- net at SW8.2 (B): now also D24.1 (K); no longer D24.2 (A)
- net at SW12.2 (B): now also D28.1 (K); no longer D28.2 (A)
- net at SW16.2 (B): now also D32.1 (K); no longer D32.2 (A)
Changed lines of the file:
@@
 	1    0    0    -1
 $EndComp
-Text GLabel 1950 3200 1    50   Input ~ 0
+Text GLabel 1900 3250 2    50   Output ~ 0
 A
-Text GLabel 2050 3200 1    50   Input ~ 0
+Text GLabel 1900 3350 2    50   Output ~ 0
 B
-Text GLabel 2150 3200 1    50   Input ~ 0
+Text GLabel 1900 3450 2    50   Output ~ 0
 C
-Text GLabel 2250 3200 1    50   Input ~ 0
+Text GLabel 1900 3550 2    50   Output ~ 0
 D
-Text GLabel 1900 5950 2    50   Output ~ 0
+Text GLabel 1900 5950 2    50   Input ~ 0
 1
-Text GLabel 1900 6050 2    50   Output ~ 0
+Text GLabel 1900 6050 2    50   Input ~ 0
 2
-Text GLabel 1900 6150 2    50   Output ~ 0
+Text GLabel 1900 6150 2    50   Input ~ 0
 3
-Text GLabel 1900 6250 2    50   Output ~ 0
+Text GLabel 1900 6250 2    50   Input ~ 0
 4
 Text Label 2150 6200 0    50   ~ 0
@@
 Text Label 2100 6650 0    50   ~ 0
 Counter2A-PWM
-Text GLabel 7500 4700 3    50   Output ~ 0
+Text GLabel 7500 4700 3    50   Input ~ 0
 D
-Text GLabel 7000 4700 3    50   Output ~ 0
+Text GLabel 7000 4700 3    50   Input ~ 0
 C
-Text GLabel 6500 4700 3    50   Output ~ 0
+Text GLabel 6500 4700 3    50   Input ~ 0
 B
-Text GLabel 6000 4700 3    50   Output ~ 0
+Text GLabel 6000 4700 3    50   Input ~ 0
 A
-Text GLabel 7950 3750 2    50   Input ~ 0
+Text GLabel 7950 3750 2    50   Output ~ 0
 4
-Text GLabel 7950 2800 2    50   Input ~ 0
+Text GLabel 7950 2800 2    50   Output ~ 0
 3
-Text GLabel 7950 1850 2    50   Input ~ 0
+Text GLabel 7950 1850 2    50   Output ~ 0
 2
-Text GLabel 7950 900  2    50   Input ~ 0
+Text GLabel 7950 900  2    50   Output ~ 0
 1
 Connection ~ 7600 3750
@@
 F 0 "D32" H 7600 4134 50  0000 C CNN
 F 1 "1N4148" H 7600 4225 50  0000 C CNN
-F 2 "Diode_SMD:D_MiniMELF_Handsoldering" H 7600 4350 50  0001 C CNN
+F 2 "Diode_SMD:D_MiniMELF" H 7600 4350 50  0001 C CNN
 F 3 "~" H 7600 4350 50  0001 C CNN
 	1    7600 4350
-	0    -1   -1   0
+	0    1    1    0
 $EndComp
 $Comp
@@
 F 0 "D28" H 7600 3184 50  0000 C CNN
 F 1 "1N4148" H 7600 3275 50  0000 C CNN
-F 2 "Diode_SMD:D_MiniMELF_Handsoldering" H 7600 3400 50  0001 C CNN
+F 2 "Diode_SMD:D_MiniMELF" H 7600 3400 50  0001 C CNN
 F 3 "~" H 7600 3400 50  0001 C CNN
 	1    7600 3400
-	0    -1   -1   0
+	0    1    1    0
 $EndComp
 $Comp
@@
 F 0 "D24" H 7600 2234 50  0000 C CNN
 F 1 "1N4148" H 7600 2325 50  0000 C CNN
-F 2 "Diode_SMD:D_MiniMELF_Handsoldering" H 7600 2450 50  0001 C CNN
+F 2 "Diode_SMD:D_MiniMELF" H 7600 2450 50  0001 C CNN
 F 3 "~" H 7600 2450 50  0001 C CNN
 	1    7600 2450
-	0    -1   -1   0
+	0    1    1    0
 $EndComp
 $Comp
@@
 F 0 "D20" H 7600 1284 50  0000 C CNN
 F 1 "1N4148" H 7600 1375 50  0000 C CNN
-F 2 "Diode_SMD:D_MiniMELF_Handsoldering" H 7600 1500 50  0001 C CNN
+F 2 "Diode_SMD:D_MiniMELF" H 7600 1500 50  0001 C CNN
 F 3 "~" H 7600 1500 50  0001 C CNN
 	1    7600 1500
-	0    -1   -1   0
+	0    1    1    0
 $EndComp
 $Comp
@@
 F 0 "D31" H 7100 4134 50  0000 C CNN
 F 1 "1N4148" H 7100 4225 50  0000 C CNN
-F 2 "Diode_SMD:D_MiniMELF_Handsoldering" H 7100 4350 50  0001 C CNN
+F 2 "Diode_SMD:D_MiniMELF" H 7100 4350 50  0001 C CNN
 F 3 "~" H 7100 4350 50  0001 C CNN
 	1    7100 4350
-	0    -1   -1   0
+	0    1    1    0
 $EndComp
 $Comp
@@
 F 0 "D27" H 7100 3184 50  0000 C CNN
 F 1 "1N4148" H 7100 3275 50  0000 C CNN
-F 2 "Diode_SMD:D_MiniMELF_Handsoldering" H 7100 3400 50  0001 C CNN
+F 2 "Diode_SMD:D_MiniMELF" H 7100 3400 50  0001 C CNN
 F 3 "~" H 7100 3400 50  0001 C CNN
 	1    7100 3400
-	0    -1   -1   0
+	0    1    1    0
 $EndComp
 $Comp
@@
 F 0 "D23" H 7100 2234 50  0000 C CNN
 F 1 "1N4148" H 7100 2325 50  0000 C CNN
-F 2 "Diode_SMD:D_MiniMELF_Handsoldering" H 7100 2450 50  0001 C CNN
+F 2 "Diode_SMD:D_MiniMELF" H 7100 2450 50  0001 C CNN
 F 3 "~" H 7100 2450 50  0001 C CNN
 	1    7100 2450
-	0    -1   -1   0
+	0    1    1    0
 $EndComp
 $Comp
@@
 F 0 "D19" H 7100 1284 50  0000 C CNN
 F 1 "1N4148" H 7100 1375 50  0000 C CNN
-F 2 "Diode_SMD:D_MiniMELF_Handsoldering" H 7100 1500 50  0001 C CNN
+F 2 "Diode_SMD:D_MiniMELF" H 7100 1500 50  0001 C CNN
 F 3 "~" H 7100 1500 50  0001 C CNN
 	1    7100 1500
-	0    -1   -1   0
+	0    1    1    0
 $EndComp
 $Comp
@@
 F 0 "D30" H 6600 4134 50  0000 C CNN
 F 1 "1N4148" H 6600 4225 50  0000 C CNN
-F 2 "Diode_SMD:D_MiniMELF_Handsoldering" H 6600 4350 50  0001 C CNN
+F 2 "Diode_SMD:D_MiniMELF" H 6600 4350 50  0001 C CNN
 F 3 "~" H 6600 4350 50  0001 C CNN
 	1    6600 4350
-	0    -1   -1   0
+	0    1    1    0
 $EndComp
 $Comp
@@
 F 0 "D26" H 6600 3184 50  0000 C CNN
 F 1 "1N4148" H 6600 3275 50  0000 C CNN
-F 2 "Diode_SMD:D_MiniMELF_Handsoldering" H 6600 3400 50  0001 C CNN
+F 2 "Diode_SMD:D_MiniMELF" H 6600 3400 50  0001 C CNN
 F 3 "~" H 6600 3400 50  0001 C CNN
 	1    6600 3400
-	0    -1   -1   0
+	0    1    1    0
 $EndComp
 $Comp
@@
 F 0 "D22" H 6600 2234 50  0000 C CNN
 F 1 "1N4148" H 6600 2325 50  0000 C CNN
-F 2 "Diode_SMD:D_MiniMELF_Handsoldering" H 6600 2450 50  0001 C CNN
+F 2 "Diode_SMD:D_MiniMELF" H 6600 2450 50  0001 C CNN
 F 3 "~" H 6600 2450 50  0001 C CNN
 	1    6600 2450
-	0    -1   -1   0
+	0    1    1    0
 $EndComp
 $Comp
@@
 F 0 "D18" H 6600 1284 50  0000 C CNN
 F 1 "1N4148" H 6600 1375 50  0000 C CNN
-F 2 "Diode_SMD:D_MiniMELF_Handsoldering" H 6600 1500 50  0001 C CNN
+F 2 "Diode_SMD:D_MiniMELF" H 6600 1500 50  0001 C CNN
 F 3 "~" H 6600 1500 50  0001 C CNN
 	1    6600 1500
-	0    -1   -1   0
+	0    1    1    0
 $EndComp
 $Comp
@@
 F 0 "D29" H 6100 4134 50  0000 C CNN
 F 1 "1N4148" H 6100 4225 50  0000 C CNN
-F 2 "Diode_SMD:D_MiniMELF_Handsoldering" H 6100 4350 50  0001 C CNN
+F 2 "Diode_SMD:D_MiniMELF" H 6100 4350 50  0001 C CNN
 F 3 "~" H 6100 4350 50  0001 C CNN
 	1    6100 4350
-	0    -1   -1   0
+	0    1    1    0
 $EndComp
 $Comp
@@
 F 0 "D25" H 6100 3184 50  0000 C CNN
 F 1 "1N4148" H 6100 3275 50  0000 C CNN
-F 2 "Diode_SMD:D_MiniMELF_Handsoldering" H 6100 3400 50  0001 C CNN
+F 2 "Diode_SMD:D_MiniMELF" H 6100 3400 50  0001 C CNN
 F 3 "~" H 6100 3400 50  0001 C CNN
 	1    6100 3400
-	0    -1   -1   0
+	0    1    1    0
 $EndComp
 $Comp
@@
 F 0 "D21" H 6100 2234 50  0000 C CNN
 F 1 "1N4148" H 6100 2325 50  0000 C CNN
-F 2 "Diode_SMD:D_MiniMELF_Handsoldering" H 6100 2450 50  0001 C CNN
+F 2 "Diode_SMD:D_MiniMELF" H 6100 2450 50  0001 C CNN
 F 3 "~" H 6100 2450 50  0001 C CNN
 	1    6100 2450
-	0    -1   -1   0
+	0    1    1    0
 $EndComp
 $Comp
@@
 F 0 "D17" H 6100 1284 50  0000 C CNN
 F 1 "1N4148" H 6100 1375 50  0000 C CNN
-F 2 "Diode_SMD:D_MiniMELF_Handsoldering" H 6100 1500 50  0001 C CNN
+F 2 "Diode_SMD:D_MiniMELF" H 6100 1500 50  0001 C CNN
 F 3 "~" H 6100 1500 50  0001 C CNN
 	1    6100 1500
-	0    -1   -1   0
+	0    1    1    0
 $EndComp
 $Comp
@@
 	2100 6200 2550 6200
 Wire Wire Line
-	1900 3250 1950 3250
-Wire Wire Line
-	1950 3250 1950 3200
-Wire Wire Line
-	1900 3350 2050 3350
-Wire Wire Line
-	2050 3350 2050 3200
-Wire Wire Line
-	1900 3450 2150 3450
-Wire Wire Line
-	2150 3450 2150 3200
-Wire Wire Line
-	1900 3550 2250 3550
-Wire Wire Line
-	2250 3550 2250 3200
-Wire Wire Line
-	1950 3250 2300 3250
-Connection ~ 1950 3250
-Wire Wire Line
-	2300 3350 2050 3350
-Connection ~ 2050 3350
-Wire Wire Line
-	2150 3450 2300 3450
-Connection ~ 2150 3450
-Wire Wire Line
-	2300 3550 2250 3550
-Connection ~ 2250 3550
-Wire Wire Line
 	7600 900  7950 900
 Wire Wire Line
@@
 	1    1300 4950
 	1    0    0    -1
-$EndComp
-Wire Wire Line
-	2750 3250 2750 3300
-Wire Wire Line
-	2700 3250 2750 3250
-$Comp
-L power:Earth #PWR04
-U 1 1 6ABA619B
-P 2750 3300
-F 0 "#PWR04" H 2750 3050 50  0001 C CNN
-F 1 "Earth" H 2750 3150 50  0001 C CNN
-F 2 "" H 2750 3300 50  0001 C CNN
-F 3 "~" H 2750 3300 50  0001 C CNN
-	1    2750 3300
-	1    0    0    -1
-$EndComp
-$Comp
-L Device:R_Network08 RN1
-U 1 1 64E45CBF
-P 2500 3650
-F 0 "RN1" V 2000 3550 50  0000 C CNN
-F 1 "100k" V 2000 3800 50  0000 C CNN
-F 2 "Resistor_THT:R_Array_SIP9" V 2975 3650 50  0001 C CNN
-F 3 "http://www.vishay.com/docs/31509/csc.pdf" H 2500 3650 50  0001 C CNN
-	1    2500 3650
-	0    1    1    0
 $EndComp
 Wire Wire Line
@@
 5v
 Wire Wire Line
-	1900 4650 2150 4650
-Wire Wire Line
-	2150 4650 2150 3650
-Wire Wire Line
-	2150 3650 2300 3650
-Wire Wire Line
-	1900 4750 2200 4750
-Wire Wire Line
-	2200 4750 2200 3750
-Wire Wire Line
-	2200 3750 2300 3750
-Wire Wire Line
-	1900 4850 2250 4850
-Wire Wire Line
-	2250 4850 2250 3850
-Wire Wire Line
-	2250 3850 2300 3850
-Wire Wire Line
 	1950 5050 1950 4550
 Connection ~ 1950 4550
@@
 NoConn ~ 1900 6450
 Wire Wire Line
-	2250 4850 2500 4850
-Connection ~ 2250 4850
-Wire Wire Line
-	2500 4750 2200 4750
-Connection ~ 2200 4750
-Wire Wire Line
-	2150 4650 2500 4650
-Connection ~ 2150 4650
-Wire Wire Line
 	700  3250 600  3250
 Wire Wire Line
 	600  3250 600  2550
 Wire Wire Line
-	600  2550 3300 2550
-Wire Wire Line
-	3300 2550 3300 4400
-Wire Wire Line
-	3300 4400 2400 4400
-Wire Wire Line
-	2400 4400 2400 4550
+	600  2550 2400 2550
 Wire Wire Line
 	2400 4550 2500 4550
@@
 	3350 5450 3450 5450
 $Comp
-L power:Earth #PWR?
+L power:Earth #PWR0101
 U 1 1 5F265FB5
 P 2550 6300
-F 0 "#PWR?" H 2550 6050 50  0001 C CNN
+F 0 "#PWR0101" H 2550 6050 50  0001 C CNN
 F 1 "Earth" H 2550 6150 50  0001 C CNN
 F 2 "" H 2550 6300 50  0001 C CNN
@@
 	0    1    1    0
 $EndComp
+Wire Wire Line
+	1900 4650 2500 4650
+Wire Wire Line
+	1900 4750 2500 4750
+Wire Wire Line
+	1900 4850 2500 4850
+Wire Wire Line
+	2400 2550 2400 4550
 $EndSCHEMATC
